File: audio_amp_lm386_mk1/audio_amp_lm386_mk1.kicad_pcb (KiCad board)
At the start: 2 copper layers, 90.1 x 57.2 mm, 22 parts, among them P1 CONN_01X03, P2 CONN_01X03, P4 CONN_01X02, U1 LM386, U2 LM386

Commit message: Commit current progress (unknown changes).
Routing:
- net Net-(RV1-Pad12): track 57.6 -> 108.9 mm
- net Net-(RV1-Pad22): track 67.1 -> 116.4 mm
- net +9V: track 91.0 -> 140.3 mm
- net Net-(C10-Pad1): track 26.0 -> 49.5 mm
- net Net-(P2-Pad1): track 27.2 -> 50.5 mm
- net Net-(C9-Pad1): track 19.9 -> 37.2 mm
- net Net-(P2-Pad3): track 17.2 -> 28.3 mm
- net Net-(C1-Pad1): track 19.3 -> 28.6 mm
- net Net-(C3-Pad1): track 13.2 -> 20.1 mm
- net Net-(C4-Pad1): track 13.2 -> 17.6 mm
Other:
- net class Default: trace_width 0.25 -> 0.5
- net class Power: trace_width 0.5 -> 1
