File: audio_amp_lm386_mk1/audio_amp_lm386_mk1.kicad_pcb (KiCad board)
At the start: 2 copper layers, 90.1 x 57.2 mm, 22 parts, among them P1 CONN_01X03, P2 CONN_01X03, P4 CONN_01X02, U1 LM386, U2 LM386

Commit message: Update progress
Other:
- board text added: "BY ANDREAS MUELLER 2017"
- board text removed: "BY ANDREAS MUELLER"
Changed lines of the file:
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@@
     )
   )
-  (gr_text "BY ANDREAS MUELLER" (at 163.83 124.46) (layer B.Cu)
+  (gr_text "BY ANDREAS MUELLER 2017" (at 160.02 124.46) (layer B.Cu)
     (effects (font (size 1.5 1.5) (thickness 0.3)) (justify mirror))
   )
