File: audio_amp_lm386_mk1/audio_amp_lm386_mk1.kicad_pcb (KiCad board)
At the start: 2 copper layers, 90.1 x 57.2 mm, 22 parts, among them P1 CONN_01X03, P2 CONN_01X03, P4 CONN_01X02, U1 LM386, U2 LM386

Commit message: Update layout, increase via size and improve routing around vias.
Parts:
- added REF**: MountingHole_3.2mm_M3_DIN965_Pad, Mounting_Holes:MountingHole_3.2mm_M3_DIN965_Pad, B.Cu at (175.3, 124.5)
- added REF**: MountingHole_3.2mm_M3_DIN965_Pad, Mounting_Holes:MountingHole_3.2mm_M3_DIN965_Pad, B.Cu at (92.7, 124.5)
- added REF**: MountingHole_3.2mm_M3_DIN965_Pad, Mounting_Holes:MountingHole_3.2mm_M3_DIN965_Pad, B.Cu at (92.7, 74.9)
- added REF**: MountingHole_3.2mm_M3_DIN965_Pad, Mounting_Holes:MountingHole_3.2mm_M3_DIN965_Pad, B.Cu at (175.3, 74.9)
- moved RV1 3.81 mm to (100.3, 110.5)
Routing:
- net Net-(RV1-Pad22): track 116.4 -> 79.0 mm
- net Net-(RV1-Pad12): track 108.9 -> 81.2 mm
- net Net-(C9-Pad1): track 37.2 -> 18.6 mm
- net Net-(C10-Pad1): track 49.5 -> 36.3 mm
