File: audio_amp_lm386_mk1/audio_amp_lm386_mk1.sch (KiCad schematic (older format))
At the start: 22 parts, among them P1 CONN_01X03, P2 CONN_01X03, P4 CONN_01X02, U1 LM386, U2 LM386

Commit message: Update layout, increase via size and improve routing around vias.
Parts:
- U1, U2: symbol LM386 -> LM386-RESCUE-audio_amp_lm386_mk1
Changed lines of the file:
@@
 EESchema Schematic File Version 2
+LIBS:audio_amp_lm386_mk1-rescue
 LIBS:power
 LIBS:device
@@
 $EndDescr
 $Comp
-L LM386 U1
+L LM386-RESCUE-audio_amp_lm386_mk1 U1
 U 1 1 58CB04A4
 P 4800 1500
@@
 $EndComp
 $Comp
-L LM386 U2
+L LM386-RESCUE-audio_amp_lm386_mk1 U2
 U 1 1 58CB050B
 P 4800 3600
