File: audio_amp_tda2030_mk1/audio_amp_tda2030_mk1.sch (KiCad schematic (older format))
At the start: 44 parts, among them P1 CONN_01X03, P2 CONN_01X02, T1 230V:2x15V, U1 TDA2030, U2 TDA2030, U3 LM7812

Commit message: Update progress
Parts:
- C13, C14: value CP -> 10u
- C15: value C -> 100n
Other:
- note added: "D1, D2, D3, D4 are for reverse voltage protection."
Changed lines of the file:
@@
 P 9400 3250
 F 0 "C13" H 9425 3350 50  0000 L CNN
-F 1 "CP" H 9425 3150 50  0000 L CNN
+F 1 "10u" H 9425 3150 50  0000 L CNN
 F 2 "" H 9438 3100 50  0001 C CNN
 F 3 "" H 9400 3250 50  0000 C CNN
@@
 P 10400 3200
 F 0 "C14" H 10425 3300 50  0000 L CNN
-F 1 "CP" H 10425 3100 50  0000 L CNN
+F 1 "10u" H 10425 3100 50  0000 L CNN
 F 2 "" H 10438 3050 50  0001 C CNN
 F 3 "" H 10400 3200 50  0000 C CNN
@@
 P 10650 3200
 F 0 "C15" H 10675 3300 50  0000 L CNN
-F 1 "C" H 10675 3100 50  0000 L CNN
+F 1 "100n" H 10675 3100 50  0000 L CNN
 F 2 "" H 10688 3050 50  0001 C CNN
 F 3 "" H 10650 3200 50  0000 C CNN
@@
 Wire Wire Line
 	10500 2350 10250 2350
+Text Notes 4050 1400 0    60   ~ 0
+D1, D2, D3, D4 are for reverse voltage protection.
 $EndSCHEMATC
