File: xcpld_demo_board/xcpld_demo_board.kicad_pcb (KiCad board)
At the start: 2 copper layers, 65.4 x 35.6 mm, 23 parts, among them P1 CONN_02X05, P2 CONN_02X05, P3 CONN_02X05, P4 CONN_02X05, P5 CONN_02X07, P6 USB_B, U1 LM317EMP, U2 XCR3064-VQ44

Commit message: Update progress
Routing:
- net Net-(C1-Pad1): track 29.0 -> 39.9 mm
- net +5V: track 0.00 -> 8.14 mm
- added copper zone on F.Cu, net COOL_PORT_EN
Changed lines of the file:
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@@
   (general
     (links 87)
-    (no_connects 2)
-    (area 73.584999 57.074999 139.778334 92.785001)
+    (no_connects 0)
+    (area 73.584999 57.074999 139.143334 92.785001)
     (thickness 1.6)
     (drawings 4)
-    (tracks 288)
+    (tracks 298)
     (zones 0)
     (modules 23)
@@
       (drillshape 1)
       (scaleselection 1)
-      (outputdirectory ""))
+      (outputdirectory output/))
   )
   (net 0 "")
@@
   (gr_line (start 139.065 92.71) (end 139.065 57.15) (angle 90) (layer Edge.Cuts) (width 0.15))
   (gr_line (start 73.66 57.15) (end 73.66 92.71) (angle 90) (layer Edge.Cuts) (width 0.15))
+  (segment (start 80.01 61.36894) (end 80.01 63.5) (width 0.2) (layer F.Cu) (net 1))
+  (segment (start 83.58886 69.61886) (end 84.836 69.61886) (width 0.2) (layer F.Cu) (net 1))
+  (segment (start 82.55 68.58) (end 83.58886 69.61886) (width 0.2) (layer F.Cu) (net 1))
+  (segment (start 82.55 66.04) (end 82.55 68.58) (width 0.2) (layer F.Cu) (net 1))
+  (segment (start 80.01 63.5) (end 82.55 66.04) (width 0.2) (layer F.Cu) (net 1))
   (segment (start 90.932 69.61886) (end 90.932 71.882) (width 0.2) (layer F.Cu) (net 1))
   (segment (start 91.694 72.644) (end 91.694 74.676) (width 0.2) (layer F.Cu) (net 1))
@@
   (segment (start 109.906 73.33) (end 109.982 73.406) (width 0.2) (layer F.Cu) (net 44))
   (via (at 109.982 73.406) (size 0.6) (drill 0.4) (layers F.Cu B.Cu) (net 44))
+  (segment (start 80.01 68.17106) (end 80.01 70.485) (width 0.35) (layer F.Cu) (net 45))
+  (segment (start 81.3109 74.2641) (end 80.30254 74.2641) (width 0.35) (layer F.Cu) (net 45))
+  (segment (start 81.915 73.66) (end 81.3109 74.2641) (width 0.35) (layer F.Cu) (net 45))
+  (segment (start 81.915 72.39) (end 81.915 73.66) (width 0.35) (layer F.Cu) (net 45))
+  (segment (start 80.01 70.485) (end 81.915 72.39) (width 0.35) (layer F.Cu) (net 45))
   (zone (net 38) (net_name COOL_PORT_EN) (layer B.Cu) (hatch edge 0.508)
     (connect_pads (clearance 0.508))
     (min_thickness 0.254)
+    (fill yes (arc_segments 16) (thermal_gap 0.508) (thermal_bridge_width 0.508))
+    (polygon
+      (pts
+        (xy 138.43 92.075) (xy 74.295 92.075) (xy 74.295 57.785) (xy 138.43 57.785) (xy 138.43 92.075)
+      )
+    )
+  )
+  (zone (net 38) (net_name COOL_PORT_EN) (layer F.Cu) (hatch edge 0.508)
+    (connect_pads (clearance 0.508))
+    (min_thickness 0.254)
